Commit message: feat: integrate hardware parameters, enable real-time odometry, and implement smart plug-and-play detection

File: src/agribot_description/urdf/agribot.urdf.xacro (robot description, xacro)
@@ -61,5 +61,5 @@
       <visual>
         <geometry>
-          <cylinder length="0.05" radius="0.1"/>
+          <cylinder length="0.04" radius="0.025"/>
         </geometry>
         <material name="black"/>
@@ -67,5 +67,5 @@
       <collision>
         <geometry>
-          <cylinder length="0.05" radius="0.1"/>
+          <cylinder length="0.04" radius="0.025"/>
         </geometry>
       </collision>
@@ -74,12 +74,12 @@
       <parent link="base_link"/>
       <child link="${prefix}_wheel"/>
-      <origin xyz="${x} ${y} -0.05" rpy="${pi/2} 0 0"/>
+      <origin xyz="${x} ${y} -0.075" rpy="${pi/2} 0 0"/>
       <axis xyz="0 0 1"/>
     </joint>
   </xacro:macro>
-  <xacro:wheel prefix="front_left" x="0.2" y="0.25"/>
-  <xacro:wheel prefix="front_right" x="0.2" y="-0.25"/>
-  <xacro:wheel prefix="rear_left" x="-0.2" y="0.25"/>
-  <xacro:wheel prefix="rear_right" x="-0.2" y="-0.25"/>
+  <xacro:wheel prefix="front_left" x="0.2" y="0.11"/>
+  <xacro:wheel prefix="front_right" x="0.2" y="-0.11"/>
+  <xacro:wheel prefix="rear_left" x="-0.2" y="0.11"/>
+  <xacro:wheel prefix="rear_right" x="-0.2" y="-0.11"/>
   <!-- Gazebo Plugins -->
   <gazebo>
@@ -90,6 +90,10 @@
       <left_joint>front_left_wheel_joint</left_joint>
       <right_joint>front_right_wheel_joint</right_joint>
-      <wheel_separation>0.5</wheel_separation>
-      <wheel_diameter>0.2</wheel_diameter>
+      <wheel_separation>0.22</wheel_separation>
+      <wheel_diameter>0.05</wheel_diameter>
+      <publish_odom>true</publish_odom>
+      <publish_odom_tf>true</publish_odom_tf>
+      <odometry_frame>odom</odometry_frame>
+      <robot_base_frame>base_link</robot_base_frame>
     </plugin>
   </gazebo>
